File: devboard/MSPM0.kicad_sch (KiCad schematic)
At the start: 66 parts, among them J1 USB_C_USB2.0, J2 SWD, J3 Conn_01x03_Pin, J4 Conn_01x02, J5 Conn_01x03_Pin, SW1 SW, SW2 SW_Push, SW3 SW, SW4 SW_Push, SW5 SW_Push, U2 AP2112K-3.3, Y2 40MHz

Commit message: clean a bit
Parts:
- TP8: value TP_UART_RX -> TP_UART_TX
- TP9: value TP_UART_TX -> TP_UART_RX
Connections:
- net +3V3: now also UNO_POWER2.4 (Pin_4)
- net 3V3_MCU: now also SW3.1; no longer UNO_POWER2.4 (Pin_4)
- net GND: now also R17.2; no longer R17.1
- net SPI_POCI: now also MCU1.16 (PB19_A1_6); no longer MCU1.56 (PA10)
- net SPI_SCLK: now also MCU1.15 (PB18_A1_5); no longer MCU1.57 (PA11)
- net UART0_RX: now also J3.3 (Pin_3), MCU1.57 (PA11), R11.2, TP9.1, UNO_DIGITAL_L2.1 (Pin_1); no longer J3.2 (Pin_2), MCU1.11 (PA18_A1_3), R12.2, SW3.1, TP8.1, UNO_DIGITAL_L2.2 (Pin_2)
- net UART0_TX: now also J3.2 (Pin_2), MCU1.56 (PA10), R12.2, TP8.1, UNO_DIGITAL_L2.2 (Pin_2); no longer J3.3 (Pin_3), MCU1.10 (PA17_A1_2), R11.2, TP9.1, UNO_DIGITAL_L2.1 (Pin_1)
- net at SW3.2: now also MCU1.11 (PA18_A1_3), R17.1; no longer R17.2
- no-connect marks 48 -> 47
Other:
- moved on the sheet: R17

Commit message: almost done with the whole schematic
Parts:
- removed R5: 10k, symbol Device:R
- removed SW1: SW, symbol Switch:SW_SPST
- D1: value LED -> RED
- D2: value LED -> GREEN
- D3: value LED -> BLUE
- TP4: value TP_GND -> TP_3V3
- Y2: now fitted
Connections:
- net +5V: no longer C2.1, C6.1, C9.1, CAN-FD1.3 (VCC), Polyfuse1.1, TP1.1, U2.1 (VIN)
- net GPIO_Button1: now also UNO_DIGITAL_L2.3 (Pin_3); no longer UNO_DIGITAL_L2.6 (Pin_6)
- net GPIO_Button2: now also UNO_DIGITAL_L2.5 (Pin_5); no longer UNO_DIGITAL_L2.7 (Pin_7)
- net GPIO_LED1: now also UNO_DIGITAL_L2.8 (Pin_8); no longer UNO_DIGITAL_L2.3 (Pin_3)
- net GPIO_LED2: now also UNO_DIGITAL_H2.1 (Pin_1); no longer UNO_DIGITAL_L2.4 (Pin_4)
- net PWM0_CCP0: now also UNO_DIGITAL_L2.4 (Pin_4); no longer UNO_DIGITAL_L2.5 (Pin_5)
- net PWM0_CCP1: now also UNO_DIGITAL_L2.6 (Pin_6)
- net PWM1_CCP0: now also UNO_DIGITAL_L2.7 (Pin_7); no longer UNO_DIGITAL_L2.8 (Pin_8)
- net PWM1_CCP1: now also UNO_DIGITAL_H2.2 (Pin_2)
- net SPI_PICO: now also UNO_DIGITAL_H2.4 (Pin_4)
- net SPI_POCI: now also UNO_DIGITAL_H2.5 (Pin_5)
- new net VBUS: C2.1, C6.1, C9.1, CAN-FD1.3 (VCC), Polyfuse1.1, TP1.1, U2.1 (VIN)
- no-connect marks 47 -> 41
Other:
- moved on the sheet: C10, C15, C16, C5, C7, J4, R10, R13, R17, R8, R9, SW4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
