File: devboard/MSPM0.kicad_sch (KiCad schematic)
At the start: 64 parts, among them J1 USB_C_USB2.0, J2 SWD, J3 Conn_01x03_Pin, J4 Conn_01x02, J5 Conn_01x03_Pin, SW2 SW_Push, SW3 SW, SW4 SW_Push, SW5 SW_Push, U2 AP2112K-3.3, Y2 40MHz

Commit message: footprints assigned
Parts:
- removed J1: USB_C_USB2.0, symbol Connector:USB_C_Receptacle_USB2.0_14P
- added USBC1: USB_C_Receptacle, Connector_USB:USB_C_Receptacle_GCT_USB4085, symbol Connector:USB_C_Receptacle_USB2.0_16P
- C1: renamed from C3; footprint (none) -> Capacitor_SMD:C_0603_1608Metric
- C10: renamed from C9; footprint (none) -> Capacitor_SMD:C_0603_1608Metric
- C11: renamed from C8; footprint (none) -> Capacitor_SMD:C_0402_1005Metric
- C12: renamed from C11; footprint (none) -> Capacitor_SMD:C_0402_1005Metric
- C13: renamed from C2; footprint (none) -> Capacitor_SMD:C_0402_1005Metric
- C14: renamed from C12; footprint (none) -> Capacitor_SMD:C_0402_1005Metric
- C2: renamed from C1; value 0.1u -> 100n; footprint (none) -> Capacitor_SMD:C_0402_1005Metric
- C3: renamed from C6; footprint (none) -> Capacitor_SMD:C_0402_1005Metric
- C4: renamed from C7; footprint (none) -> Capacitor_SMD:C_0402_1005Metric
- C5: value 0.47u -> 470n; footprint (none) -> Capacitor_SMD:C_0402_1005Metric
- C6: renamed from C4; footprint (none) -> Capacitor_SMD:C_0402_1005Metric
- C7: renamed from C15; footprint (none) -> Capacitor_SMD:C_0402_1005Metric
- C8: renamed from C16; footprint (none) -> Capacitor_SMD:C_0402_1005Metric
- C9: renamed from C10; footprint (none) -> Capacitor_SMD:C_0402_1005Metric
- D1: footprint (none) -> LED_SMD:LED_0603_1608Metric
- D2: renamed from D3; footprint (none) -> LED_SMD:LED_0603_1608Metric
- D3: renamed from D2; footprint (none) -> LED_SMD:LED_0603_1608Metric
- J2: renamed from J3; footprint (none) -> Connector_PinHeader_2.54mm:PinHeader_1x03_P2.54mm_Vertical
- J3: renamed from J2; footprint (none) -> Connector_PinHeader_1.27mm:PinHeader_2x05_P1.27mm_Vertical
- J5: footprint (none) -> Connector_PinHeader_2.54mm:PinHeader_1x03_P2.54mm_Vertical
- JP1: footprint (none) -> Jumper:Jumper_Harwin_S1621_P10.9mm
- Polyfuse1: footprint (none) -> Fuse:Fuse_1206_3216Metric
- R1: renamed from R8; footprint (none) -> Resistor_SMD:R_0402_1005Metric
- R10: renamed from R17; footprint (none) -> Resistor_SMD:R_0402_1005Metric
- R11: renamed from R9; footprint (none) -> Resistor_SMD:R_0402_1005Metric
- R12: renamed from R10; footprint (none) -> Resistor_SMD:R_0402_1005Metric
- R13: renamed from R11; footprint (none) -> Resistor_SMD:R_0402_1005Metric
- R14: renamed from R12; footprint (none) -> Resistor_SMD:R_0402_1005Metric
- R15: renamed from R6; footprint (none) -> Resistor_SMD:R_0402_1005Metric
- R16: renamed from R7; footprint (none) -> Resistor_SMD:R_0402_1005Metric
- R17: renamed from R13; footprint (none) -> Resistor_SMD:R_0402_1005Metric
- R18: renamed from R14; footprint (none) -> Resistor_SMD:R_0402_1005Metric
- R2: renamed from R1; footprint (none) -> Resistor_SMD:R_0402_1005Metric
- R3: renamed from R19; footprint (none) -> Resistor_SMD:R_0402_1005Metric
- R4: renamed from R2; footprint (none) -> Resistor_SMD:R_0402_1005Metric
- R5: renamed from R18; footprint (none) -> Resistor_SMD:R_0402_1005Metric
- R6: renamed from R3; footprint (none) -> Resistor_SMD:R_0402_1005Metric
- R7: renamed from R4; footprint (none) -> Resistor_SMD:R_0402_1005Metric
- R8: renamed from R16; footprint (none) -> Resistor_SMD:R_0402_1005Metric
- R9: renamed from R15; footprint (none) -> Resistor_SMD:R_0402_1005Metric
- SW1: renamed from SW2; footprint (none) -> Button_Switch_THT:SW_PUSH_6mm
- SW2: renamed from SW5; footprint (none) -> Button_Switch_THT:SW_PUSH_6mm_H7.3mm
- SW3: renamed from SW4; footprint (none) -> Button_Switch_THT:SW_PUSH_6mm_H7.3mm
- SW4: renamed from SW3; footprint (none) -> Button_Switch_THT:SW_PUSH_6mm
- TP1: renamed from TP4; footprint (none) -> TestPoint:TestPoint_Pad_D1.5mm
- TP2: renamed from TP1; footprint (none) -> TestPoint:TestPoint_Pad_D1.5mm
- TP3: renamed from TP2; footprint (none) -> TestPoint:TestPoint_Pad_D1.5mm
- TP4: renamed from TP3; footprint (none) -> TestPoint:TestPoint_Pad_D1.5mm
- TP5: renamed from TP7; footprint (none) -> TestPoint:TestPoint_Pad_D1.5mm
- TP6: renamed from TP5; footprint (none) -> TestPoint:TestPoint_Pad_D1.5mm
- TP7: renamed from TP6; footprint (none) -> TestPoint:TestPoint_Pad_D1.5mm
- TP8, TP9: footprint (none) -> TestPoint:TestPoint_Pad_D1.5mm
- renumbered J4 to J1, U2 to U1, UNO_ANALOG2 to UNO_ANALOG1, UNO_DIGITAL_H2 to UNO_DIGITAL_H1, UNO_DIGITAL_L2 to UNO_DIGITAL_L1, UNO_POWER2 to UNO_POWER1, Y2 to Y1
Connections:
- net +5V is gone; now on net VBUS: U1.3 (EN), UNO_POWER1.5 (Pin_5)
- net +3V3: no longer C4.1, J1.1 (Pin_1), R1.2, TP3.1, U1.5 (VOUT)
- net GND: now also USBC1.A1 (GND), USBC1.A12 (GND), USBC1.B1 (GND), USBC1.B12 (GND), USBC1.SH (SHIELD)
- net PWR_LED0_K: now reaches D1.2 (A), R1.1
- net at R15.2: now also USBC1.A5 (CC1)
- net at Polyfuse1.2: now also USBC1.A4 (VBUS), USBC1.A9 (VBUS), USBC1.B4 (VBUS), USBC1.B9 (VBUS)
- net at USB-UART1.5 (UD+): now also USBC1.A6 (D+), USBC1.B6 (D+)
- net at USB-UART1.6 (UD-): now also USBC1.A7 (D-), USBC1.B7 (D-)
- net at R16.2: now also USBC1.B5 (CC2)
- new net: C4.1, J1.1 (Pin_1), R1.2, TP3.1, U1.5 (VOUT)
- no-connect marks 41 -> 43
Other:
- note added: "CAN-FD"
- note added: "Crystal"
- note added: "LDO 5V -> 3.3V"
- note added: "Power Flags"
- note added: "SWD Debug"
- note added: "UNO Headers"
- note added: "USB Type-C -> USB-UART Bridge"
- note added: "USER LEDs & Buttons"

Commit message: started layout, but <bruhh> i forgot i couldnt edit layout of mcu
Connections:
- net 3V3_MCU: now also MCU1.1 (VDD); no longer MCU1.40 (VDD)
- net GND: now also MCU1.2 (VSS); no longer MCU1.41 (VSS)
- net GPIO_LED1: now also MCU1.40 (PB13); no longer MCU1.1 (PB13)
- net GPIO_LED2: now also MCU1.41 (PB14); no longer MCU1.2 (PB14)
- net NRST: now also MCU1.14 (RST_N); no longer MCU1.38 (RST_N)
- net PWR_LED1_K: now reaches D3.2 (A), R9.2
- net PWR_LED2_K: now reaches D2.2 (A), R8.2
Other:
- moved on the sheet: C1
Changed lines of the file:
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@@
 	)
 	(junction
-		(at 99.06 21.59)
-		(diameter 0)
-		(color 0 0 0 0)
-	)
-	(junction
 		(at 85.09 90.17)
 		(diameter 0)
@@
 	)
 	(junction
-		(at 99.06 29.21)
+		(at 228.6 114.3)
 		(diameter 0)
 		(color 0 0 0 0)
 	)
 	(junction
-		(at 228.6 114.3)
+		(at 255.27 41.91)
 		(diameter 0)
 		(color 0 0 0 0)
 	)
 	(junction
-		(at 255.27 41.91)
+		(at 100.33 29.21)
 		(diameter 0)
 		(color 0 0 0 0)
@@
 	)
 	(junction
+		(at 100.33 21.59)
+		(diameter 0)
+		(color 0 0 0 0)
+	)
+	(junction
 		(at 215.9 124.46)
 		(diameter 0)
@@
 	(wire
 		(pts
+			(xy 100.33 29.21) (xy 109.22 29.21)
+		)
+		(stroke
+			(width 0)
+			(type default)
+		)
+	)
+	(wire
+		(pts
 			(xy 215.9 121.92) (xy 215.9 123.19)
 		)
@@
 	(wire
 		(pts
+			(xy 100.33 21.59) (xy 109.22 21.59)
+		)
+		(stroke
+			(width 0)
+			(type default)
+		)
+	)
+	(wire
+		(pts
 			(xy 72.39 58.42) (xy 74.93 58.42)
 		)
@@
 	(wire
 		(pts
-			(xy 91.44 21.59) (xy 99.06 21.59)
+			(xy 91.44 21.59) (xy 100.33 21.59)
 		)
 		(stroke
@@
 	(wire
 		(pts
-			(xy 203.2 67.31) (xy 201.93 67.31)
+			(xy 201.93 67.31) (xy 204.47 67.31)
 		)
 		(stroke
@@
 	(wire
 		(pts
-			(xy 203.2 59.69) (xy 201.93 59.69)
+			(xy 207.01 59.69) (xy 201.93 59.69)
 		)
 		(stroke
@@
 	(wire
 		(pts
-			(xy 99.06 29.21) (xy 109.22 29.21)
+			(xy 99.06 29.21) (xy 100.33 29.21)
 		)
 		(stroke
@@
 	(wire
 		(pts
-			(xy 210.82 67.31) (xy 213.36 67.31)
+			(xy 212.09 67.31) (xy 214.63 67.31)
 		)
 		(stroke
@@
 	(wire
 		(pts
-			(xy 99.06 21.59) (xy 109.22 21.59)
-		)
-		(stroke
-			(width 0)
-			(type default)
-		)
-	)
-	(wire
-		(pts
 			(xy 203.2 41.91) (xy 194.31 41.91)
 		)
@@
 	(wire
 		(pts
-			(xy 210.82 59.69) (xy 213.36 59.69)
+			(xy 214.63 59.69) (xy 217.17 59.69)
 		)
 		(stroke
@@
 	)
 	(label "PWR_LED1_K"
-		(at 213.36 67.31 0)
+		(at 203.2 67.31 270)
 		(effects
 			(font
 				(size 1.27 1.27)
 			)
-			(justify left bottom)
+			(justify right bottom)
 		)
 	)
@@
 	)
 	(label "PWR_LED2_K"
-		(at 213.36 59.69 0)
+		(at 205.74 59.69 270)
 		(effects
 			(font
 				(size 1.27 1.27)
 			)
-			(justify left bottom)
+			(justify right bottom)
 		)
 	)
@@
 	(symbol
 		(lib_id "Device:LED")
-		(at 207.01 67.31 180)
+		(at 208.28 67.31 180)
 		(unit 1)
 		(body_style 1)
@@
 		(dnp no)
 		(property "Reference" "D3"
-			(at 208.5975 59.69 0)
+			(at 209.8675 59.69 0)
 			(hide yes)
 			(show_name no)
@@
 		)
 		(property "Value" "GREEN"
-			(at 208.534 70.104 0)
+			(at 209.804 70.104 0)
 			(show_name no)
 			(do_not_autoplace no)
@@
 		)
 		(property "Footprint" "LED_SMD:LED_0603_1608Metric"
-			(at 207.01 67.31 0)
+			(at 208.28 67.31 0)
 			(hide yes)
 			(show_name no)
@@
 		)
 		(property "Datasheet" ""
-			(at 207.01 67.31 0)
+			(at 208.28 67.31 0)
 			(hide yes)
 			(show_name no)
@@
 		)
 		(property "Description" "Light emitting diode"
-			(at 207.01 67.31 0)
+			(at 208.28 67.31 0)
 			(hide yes)
 			(show_name no)
@@
 		)
 		(property "Sim.Pins" "1=K 2=A"
-			(at 207.01 67.31 0)
+			(at 208.28 67.31 0)
 			(hide yes)
 			(show_name no)
@@
 	(symbol
 		(lib_id "Device:C")
-		(at 99.06 25.4 0)
+		(at 100.33 25.4 0)
 		(unit 1)
 		(body_style 1)
@@
 		(in_pos_files yes)
 		(dnp no)
-		(fields_autoplaced yes)
 		(property "Reference" "C1"
-			(at 102.87 24.1299 0)
+			(at 102.616 24.13 0)
 			(show_name no)
 			(do_not_autoplace no)
@@
 		)
 		(property "Value" "10u"
-			(at 102.87 26.6699 0)
+			(at 102.616 26.67 0)
 			(show_name no)
 			(do_not_autoplace no)
@@
 		)
 		(property "Footprint" "Capacitor_SMD:C_0603_1608Metric"
-			(at 100.0252 29.21 0)
+			(at 101.2952 29.21 0)
 			(hide yes)
 			(show_name no)
@@
 		)
 		(property "Datasheet" ""
-			(at 99.06 25.4 0)
+			(at 100.33 25.4 0)
 			(hide yes)
 			(show_name no)
@@
 		)
 		(property "Description" "Unpolarized capacitor"
-			(at 99.06 25.4 0)
+			(at 100.33 25.4 0)
 			(hide yes)
 			(show_name no)
@@
 	(symbol
 		(lib_id "power:GND")
-		(at 213.36 59.69 0)
+		(at 217.17 59.69 0)
 		(unit 1)
 		(body_style 1)
@@
 		(fields_autoplaced yes)
 		(property "Reference" "#PWR021"
-			(at 213.36 66.04 0)
+			(at 217.17 66.04 0)
 			(hide yes)
 			(show_name no)
@@
 		)
 		(property "Value" "GND"
-			(at 213.36 64.77 0)
+			(at 217.17 64.77 0)
 			(hide yes)
 			(show_name no)
@@
 		)
 		(property "Footprint" ""
-			(at 213.36 59.69 0)
+			(at 217.17 59.69 0)
 			(hide yes)
 			(show_name no)
@@
 		)
 		(property "Datasheet" ""
-			(at 213.36 59.69 0)
+			(at 217.17 59.69 0)
 			(hide yes)
 			(show_name no)
@@
 		)
 		(property "Description" "Power symbol creates a global label with name \"GND\" , ground"
-			(at 213.36 59.69 0)
+			(at 217.17 59.69 0)
 			(hide yes)
 			(show_name no)
@@
 	(symbol
 		(lib_id "power:GND")
-		(at 213.36 67.31 0)
+		(at 214.63 67.31 0)
 		(unit 1)
 		(body_style 1)
@@
 		(fields_autoplaced yes)
 		(property "Reference" "#PWR022"
-			(at 213.36 73.66 0)
+			(at 214.63 73.66 0)
 			(hide yes)
 			(show_name no)
@@
 		)
 		(property "Value" "GND"
-			(at 213.36 72.39 0)
+			(at 214.63 72.39 0)
 			(hide yes)
 			(show_name no)
@@
 		)
 		(property "Footprint" ""
-			(at 213.36 67.31 0)
+			(at 214.63 67.31 0)
 			(hide yes)
 			(show_name no)
@@
 		)
 		(property "Datasheet" ""
-			(at 213.36 67.31 0)
+			(at 214.63 67.31 0)
 			(hide yes)
 			(show_name no)
@@
 		)
 		(property "Description" "Power symbol creates a global label with name \"GND\" , ground"
-			(at 213.36 67.31 0)
+			(at 214.63 67.31 0)
 			(hide yes)
 			(show_name no)
@@
 	(symbol
 		(lib_id "Device:LED")
-		(at 207.01 59.69 180)
+		(at 210.82 59.69 180)
 		(unit 1)
 		(body_style 1)
@@
 		(dnp no)
 		(property "Reference" "D2"
-			(at 208.5975 52.07 0)
+			(at 212.4075 52.07 0)
 			(hide yes)
 			(show_name no)
@@
 		)
 		(property "Value" "BLUE"
-			(at 208.534 62.484 0)
+			(at 212.344 62.484 0)
 			(show_name no)
 			(do_not_autoplace no)
@@
 		)
 		(property "Footprint" "LED_SMD:LED_0603_1608Metric"
-			(at 207.01 59.69 0)
+			(at 210.82 59.69 0)
 			(hide yes)
 			(show_name no)
@@
 		)
 		(property "Datasheet" ""
-			(at 207.01 59.69 0)
+			(at 210.82 59.69 0)
 			(hide yes)
 			(show_name no)
@@
 		)
 		(property "Description" "Light emitting diode"
-			(at 207.01 59.69 0)
+			(at 210.82 59.69 0)
 			(hide yes)
 			(show_name no)
@@
 		)
 		(property "Sim.Pins" "1=K 2=A"
-			(at 207.01 59.69 0)
+			(at 210.82 59.69 0)
 			(hide yes)
 			(show_name no)
