File: devboard/MSPM0.kicad_pcb (KiCad board)
At the start: 2 copper layers, 64 parts, among them J1 Conn_01x02, J2 Conn_01x03_Pin, J5 Conn_01x03_Pin, SW1 SW_Push, SW2 SW_Push, SW3 SW_Push, SW4 SW, U1 AP2112K-3.3, Y1 40MHz

Commit message: ok, fixed the footprint, and placed the main components onto the board
Parts:
- added REF**: Arduino_UNO_R3_WithMountingHoles, Module:Arduino_UNO_R3_WithMountingHoles, F.Cu at (185.8, 34.9)
- moved C10 123.8 mm to (217.8, 62.5), turned to -90 degrees
- moved R18 109.8 mm to (214.3, 43.8), turned to 90 degrees
- moved R17 107.2 mm to (212.6, 43.7), turned to -90 degrees
- moved J1 100.6 mm to (210.0, 72.5)
- moved J5 92.3 mm to (209.3, 49.2), turned to 180 degrees
- moved C14 91.9 mm to (213.3, 46.0), turned to -90 degrees
- moved Polyfuse1 86.8 mm to (216.2, 66.8)
- moved C12 81.5 mm to (202.6, 46.0)
- moved JP1 78.3 mm to (206.3, 40.2)
- moved C13 77.8 mm to (201.1, 51.7), turned to 180 degrees
- moved C9 42.2 mm to (195.3, 45.8), turned to 180 degrees
- moved R11 42.2 mm to (198.1, 46.2), turned to -90 degrees
- moved USBC1 41.1 mm to (219.7, 62.8), turned to 90 degrees
- moved USB-UART1 39.8 mm to (212.5, 55.2), turned to 90 degrees
- moved J3 39.2 mm to (195.8, 48.0), turned to -90 degrees
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- renumbered SWD to J3
Connections:
- MCU1 pad 1: /3V3_MCU -> /GPIO_LED1
- MCU1 pad 14: /NRST -> unconnected-(MCU1-PB17_A1_4-Pad14)
- MCU1 pad 2: GND -> /GPIO_LED2
- MCU1 pad 38: unconnected-(MCU1-PB17_A1_4-Pad38) -> /NRST
- MCU1 pad 40: /GPIO_LED1 -> /3V3_MCU
- MCU1 pad 41: /GPIO_LED2 -> GND
Routing:
- net Net-(USB-UART1-UD-): track 5.76 -> 6.47 mm
- net Net-(USB-UART1-UD+): track 7.38 -> 8.09 mm
